Commit message: kleine aanpassingen

File: description/robot.urdf.xacro (robot description, xacro)
@@ -2,3 +2,4 @@
 <robot xmlns:xacro="http://www.ros.org/wiki/xacro"  name="robot">
    <xacro:include filename="robotcore.xacro"/>
+   <xacro:include filename="gazebo_control.xacro"/>
 </robot>

File: description/robotcore.xacro (robot description, xacro)
@@ -5,5 +5,5 @@
     <parent link="base_footprint"/>
     <child link="base_link"/>
-    <origin xyz="0 0 0.1"/>
+    <origin xyz="0 0 0.15"/>
   </joint>
   <link name="base_link">
@@ -55,4 +55,8 @@
         </inertial>
     </link>
+    <gazebo reference="caster_back">
+        <mu1 value= "0.001"/>
+        <mu2 value="0.001"/>
+        </gazebo>
   <!-- Laser Scanner -->
   <joint name="laser_joint" type="fixed">

Commit message: bruh

File: description/robot.urdf.xacro (robot description, xacro)
@@ -1,5 +1,6 @@
 <?xml version="1.0"?>
-<robot xmlns:xacro="http://www.ros.org/wiki/xacro"  name="robot">
+<robot xmlns:xacro="http://www.ros.org/wiki/xacro"  name="my_bot">
    <xacro:include filename="robotcore.xacro"/>
    <xacro:include filename="gazebo_control.xacro"/>
+   <xacro:include filename="lidar.xacro"/>
 </robot>

File: description/robotcore.xacro (robot description, xacro)
@@ -59,12 +59,3 @@
         <mu2 value="0.001"/>
         </gazebo>
-  <!-- Laser Scanner -->
-  <joint name="laser_joint" type="fixed">
-    <parent link="base_link"/>
-    <child link="laser_link"/>
-    <origin xyz="0.2 0 0.1"/>
-  </joint>
-  <link name="laser_link">
-    <visual><geometry><cylinder length="0.05" radius="0.05"/></geometry></visual>
-  </link>
 </robot>
